File: Hardware/TH8200Control.sch (KiCad schematic (older format))
At the start: 39 parts, among them J1 Mains, J2 Heater Relay, J3 Motor, Q1 BC817, Q2 SFH 300, Q3 BC817, Q4 BC817, T1 BV EI 306 3601, U1 CNY17-3, U2 CNY17-3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

Commit message: Add ISP header
Parts:
- added J4: ISP, Pin_Headers:Pin_Header_Straight_SMT_02x03, symbol conn:CONN_02X03
Connections:
- net +5V: now also J4.2 (P2)
- net GND: now also J4.6 (P6)
- net ISP_RESET: now reaches R9.1, U4.29 ((PCINT14/~RESET~)PC6)
- net ISP_RESET: now also J4.5 (P5)
- net ISP_COPI: now reaches U4.15 ((PCINT3/OC2A/MOSI)PB3)
- net ISP_COPI: now also J4.4 (P4)
- net ISP_CIPO: now reaches U4.16 ((PCINT4/MISO)PB4)
- net ISP_CIPO: now also J4.1 (P1)
- net ISP_SCK: now reaches U4.17 ((PCINT5/SCK)PB5)
- net ISP_SCK: now also J4.3 (P3)
- no-connect marks 17 -> 14
Other:
- moved on the sheet: R9
Changed lines of the file:
@@
 Sheet 1 1
 Title "Control board for Siemens TH8200 hand dryer"
-Date "2020-07-20"
+Date "2020-07-22"
 Rev "1.0"
 Comp "xatLabs"
@@
 L device:R R9
 U 1 1 5F230178
-P 10400 5200
-F 0 "R9" H 10330 5154 50  0000 R CNN
-F 1 "4.7k" H 10330 5245 50  0000 R CNN
-F 2 "Resistors_SMD:R_0603" V 10330 5200 50  0001 C CNN
-F 3 "~" H 10400 5200 50  0001 C CNN
-	1    10400 5200
+P 10250 5200
+F 0 "R9" H 10180 5154 50  0000 R CNN
+F 1 "4.7k" H 10180 5245 50  0000 R CNN
+F 2 "Resistors_SMD:R_0603" V 10180 5200 50  0001 C CNN
+F 3 "~" H 10250 5200 50  0001 C CNN
+	1    10250 5200
 	-1   0    0    1
 $EndComp
@@
 L power:+5V #PWR020
 U 1 1 5F2C1539
-P 10400 4950
-F 0 "#PWR020" H 10400 4800 50  0001 C CNN
-F 1 "+5V" H 10415 5123 50  0000 C CNN
-F 2 "" H 10400 4950 50  0001 C CNN
-F 3 "" H 10400 4950 50  0001 C CNN
-	1    10400 4950
-	1    0    0    -1
-$EndComp
-Wire Wire Line
-	10400 4950 10400 5050
-Wire Wire Line
-	10050 5450 10400 5450
-Wire Wire Line
-	10400 5450 10400 5350
+P 10250 4950
+F 0 "#PWR020" H 10250 4800 50  0001 C CNN
+F 1 "+5V" H 10265 5123 50  0000 C CNN
+F 2 "" H 10250 4950 50  0001 C CNN
+F 3 "" H 10250 4950 50  0001 C CNN
+	1    10250 4950
+	1    0    0    -1
+$EndComp
+Wire Wire Line
+	10250 4950 10250 5050
+Wire Wire Line
+	10050 5450 10250 5450
+Wire Wire Line
+	10250 5450 10250 5350
 $Comp
 L device:C C3
@@
 	10050 4000 10150 4000
 NoConn ~ 10050 4200
-NoConn ~ 10050 4300
-NoConn ~ 10050 4400
-NoConn ~ 10050 4500
 NoConn ~ 10050 4850
 NoConn ~ 10050 4950
@@
 	0    -1   -1   0
 $EndComp
+$Comp
+L conn:CONN_02X03 J4
+U 1 1 5F18D141
+P 7100 6150
+F 0 "J4" H 7100 6465 50  0000 C CNN
+F 1 "ISP" H 7100 6374 50  0000 C CNN
+F 2 "Pin_Headers:Pin_Header_Straight_SMT_02x03" H 7100 4950 50  0001 C CNN
+F 3 "" H 7100 4950 50  0000 C CNN
+	1    7100 6150
+	1    0    0    -1
+$EndComp
+Text GLabel 10350 5450 2    50   Input ~ 0
+ISP_RESET
+Wire Wire Line
+	10250 5450 10350 5450
+Connection ~ 10250 5450
+Text GLabel 10150 4400 2    50   Input ~ 0
+ISP_CIPO
+Text GLabel 10150 4300 2    50   Output ~ 0
+ISP_COPI
+Text GLabel 10150 4500 2    50   BiDi ~ 0
+ISP_SCK
+Wire Wire Line
+	10050 4300 10150 4300
+Wire Wire Line
+	10150 4400 10050 4400
+Wire Wire Line
+	10050 4500 10150 4500
+Text GLabel 7450 6150 2    50   Input ~ 0
+ISP_COPI
+Text GLabel 6750 6050 0    50   Output ~ 0
+ISP_CIPO
+Text GLabel 6750 6150 0    50   BiDi ~ 0
+ISP_SCK
+Text GLabel 6750 6250 0    50   Output ~ 0
+ISP_RESET
+$Comp
+L power:+5V #PWR0101
+U 1 1 5F1ACFF4
+P 7450 5950
+F 0 "#PWR0101" H 7450 5800 50  0001 C CNN
+F 1 "+5V" H 7465 6123 50  0000 C CNN
+F 2 "" H 7450 5950 50  0001 C CNN
+F 3 "" H 7450 5950 50  0001 C CNN
+	1    7450 5950
+	1    0    0    -1
+$EndComp
+$Comp
+L power:GND #PWR0102
+U 1 1 5F1AD082
+P 7450 6350
+F 0 "#PWR0102" H 7450 6100 50  0001 C CNN
+F 1 "GND" H 7455 6177 50  0000 C CNN
+F 2 "" H 7450 6350 50  0001 C CNN
+F 3 "" H 7450 6350 50  0001 C CNN
+	1    7450 6350
+	1    0    0    -1
+$EndComp
+Wire Wire Line
+	7450 6350 7450 6250
+Wire Wire Line
+	7450 6250 7350 6250
+Wire Wire Line
+	7350 6150 7450 6150
+Wire Wire Line
+	7450 5950 7450 6050
+Wire Wire Line
+	7450 6050 7350 6050
+Wire Wire Line
+	6750 6050 6850 6050
+Wire Wire Line
+	6750 6150 6850 6150
+Wire Wire Line
+	6750 6250 6850 6250
 $EndSCHEMATC

Commit message: Fix polarity of C1
Connections:
- net +12V: now also C1.1; no longer C1.2
- net GND: now also C1.2; no longer C1.1
Changed lines of the file:
@@
 Sheet 1 1
 Title "Control board for Siemens TH8200 hand dryer"
-Date "2020-07-22"
-Rev "1.0"
+Date "2020-07-29"
+Rev "1.1"
 Comp "xatLabs"
 Comment1 "Julian Metzler"
@@
 F 3 "~" H 4500 1600 50  0001 C CNN
 	1    4500 1600
-	1    0    0    1
+	1    0    0    -1
 $EndComp
 Wire Wire Line
